Commit message: reanalyzed and inputed new inertias for arm, body, and rotors

File: pybullet/urdf/pelican.urdf (robot description, URDF)
Before this commit: robot pelican, 9 links, 8 joints
Links:
- link back_arm: mass None -> 0.098; geometry visual cylinder length=0.15 radius=0.01
- link back_rotor: mass 0.1 -> 0.009; geometry collision cylinder length=0.01 radius=0.128; visual cylinder length=0.01 radius=0.128
- link base_link: mass 1.0 -> 0.217
- link front_arm: mass None -> 0.098; geometry visual cylinder length=0.15 radius=0.01
- link front_rotor: mass 0.1 -> 0.009; geometry collision cylinder length=0.01 radius=0.128; visual cylinder length=0.01 radius=0.128
- link left_arm: mass None -> 0.098; geometry visual cylinder length=0.15 radius=0.01
- link left_rotor: mass 0.1 -> 0.009; geometry collision cylinder length=0.01 radius=0.128; visual cylinder length=0.01 radius=0.128
- link right_arm: mass None -> 0.098; geometry visual cylinder length=0.15 radius=0.01
- link right_rotor: mass 0.1 -> 0.009; geometry collision cylinder length=0.01 radius=0.128; visual cylinder length=0.01 radius=0.128
Joints:
- joint back_arm_joint: origin xyz=-0.105 0 0 rpy=0 0 0 -> xyz=-0.060 0 0 rpy=0 0 0
- joint back_rotor_joint: origin xyz=-0.21 0 0.05 rpy=0 0 0 -> xyz=-0.15 0 0.05 rpy=0 0 0; parent base_link -> back_arm
- joint front_arm_joint: origin xyz=0.105 0 0 rpy=0 0 0 -> xyz=0.060 0 0 rpy=0 0 0
- joint front_rotor_joint: origin xyz=0.21 0 0.05 rpy=0 0 0 -> xyz=0.15 0 0.05 rpy=0 0 0; parent base_link -> front_arm
- joint left_arm_joint: origin xyz=0 0.105 0 rpy=0 0 0 -> xyz=0 0.060 0 rpy=0 0 0
- joint left_rotor_joint: origin xyz=0 0.21 0.05 rpy=0 0 0 -> xyz=0 0.15 0.05 rpy=0 0 0; parent base_link -> left_arm
- joint right_arm_joint: origin xyz=0 -0.105 0 rpy=0 0 0 -> xyz=0 -0.060 0 rpy=0 0 0
- joint right_rotor_joint: origin xyz=0 -0.21 0.05 rpy=0 0 0 -> xyz=0 -0.15 0.05 rpy=0 0 0; parent base_link -> right_arm
